File: PWM-Buck/layout/PWM Buck V1.brd (EAGLE design)
At the start: 112.4 x 63.5 mm, 58 parts, among them IC1 AT-MEGA8-P, IC2 LP2950ACZ-3.0, T2 BC547, T3 BC338, T4 BC328, T5 IRF4905, T6 IRF4905, X1 057-010-0

Commit message: minor changes
Parts:
- added R3: 5k, 0_Eigene:R_10
Connections:
- net GND: now also R3.2
- net PWM: now also R3.1
Routing:
- net PWM: track 89.8 -> 90.8 mm
Changed lines of the file:
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@@
 <element name="S5" library="0_Eigene" package="RIA-183-05" value="" x="20.574" y="57.023"/>
 <element name="IC2" library="v-reg" package="TO92" value="LP2950ACZ-3.0" x="49.022" y="57.15" rot="R270"/>
+<element name="R3" library="0_Eigene" package="R_10" value="5k" x="42.291" y="19.177"/>
 </elements>
 <signals>
@@
 <via x="100.203" y="15.621" extent="1-16" drill="3.2" diameter="6.4516" shape="octagon"/>
 <contactref element="IC2" pad="2"/>
+<contactref element="R3" pad="2"/>
 </signal>
 <signal name="VCC">
@@
 <wire x1="37.846" y1="13.97" x2="40.132" y2="11.684" width="0.6096" layer="16"/>
 <wire x1="40.132" y1="11.684" x2="40.132" y2="8.255" width="0.6096" layer="16"/>
-<wire x1="40.132" y1="8.255" x2="39.751" y2="7.874" width="0.6096" layer="16"/>
-<wire x1="39.751" y1="7.874" x2="39.624" y2="7.747" width="0.6096" layer="16"/>
+<wire x1="40.132" y1="8.255" x2="39.624" y2="7.747" width="0.6096" layer="16"/>
 <wire x1="39.624" y1="7.747" x2="39.624" y2="3.81" width="0.4064" layer="16"/>
 <wire x1="39.624" y1="3.81" x2="39.751" y2="3.683" width="0.254" layer="16"/>
@@
 <wire x1="8.001" y1="19.558" x2="8.763" y2="20.32" width="0.6096" layer="16"/>
 <wire x1="8.763" y1="20.32" x2="8.763" y2="26.797" width="0.6096" layer="16"/>
+<contactref element="R3" pad="1"/>
+<wire x1="37.846" y1="19.558" x2="37.211" y2="19.558" width="0.4064" layer="16"/>
+<wire x1="37.211" y1="19.558" x2="37.211" y2="19.177" width="0.4064" layer="16"/>
 </signal>
 <signal name="N$7">
