File: PWM-Buck/layout/PWM Buck V1.sch (EAGLE design)
At the start: 57 parts, among them IC1 AT-MEGA8-P, IC2 LP2950ACZ-3.0, T2 BC547, T3 BC338, T4 BC328, T5 IRF4905, T6 IRF4905, X1 057-010-0

Commit message: minor changes
Parts:
- added R3: 5k, 0_Eigene:R_10
Connections:
- net GND: now also R3.2
- net PWM: now also R3.1
Changed lines of the file:
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@@
 <part name="S5" library="0_Eigene" deviceset="CON-RIA-183-05" device=""/>
 <part name="IC2" library="v-reg" deviceset="LP2950?*" device="ACZ" technology="-3.0"/>
+<part name="R3" library="0_Eigene" deviceset="R_10" device="" value="5k"/>
+<part name="GND2" library="supply1" deviceset="GND" device=""/>
 </parts>
 <sheets>
@@
 <instance part="S5" gate="5" x="104.14" y="22.86" rot="R180"/>
 <instance part="IC2" gate="G$1" x="116.84" y="93.98"/>
+<instance part="R3" gate="G$1" x="144.78" y="68.58" smashed="yes" rot="R270">
+<attribute name="NAME" x="143.51" y="66.04" size="1.778" layer="95" rot="R90"/>
+<attribute name="VALUE" x="147.32" y="66.04" size="1.27" layer="96" rot="R90"/>
+</instance>
+<instance part="GND2" gate="1" x="144.78" y="60.96" smashed="yes">
+<attribute name="VALUE" x="142.24" y="58.42" size="1.778" layer="96"/>
+</instance>
 </instances>
 <busses>
@@
 <junction x="193.04" y="-68.58"/>
 </segment>
+<segment>
+<pinref part="R3" gate="G$1" pin="2"/>
+<pinref part="GND2" gate="1" pin="GND"/>
+</segment>
 </net>
 <net name="VCC" class="0">
@@
 <wire x1="121.92" y1="35.56" x2="121.92" y2="53.34" width="0.1524" layer="91"/>
 <wire x1="121.92" y1="53.34" x2="121.92" y2="73.66" width="0.1524" layer="91"/>
-<wire x1="121.92" y1="73.66" x2="147.32" y2="73.66" width="0.1524" layer="91"/>
+<wire x1="121.92" y1="73.66" x2="144.78" y2="73.66" width="0.1524" layer="91"/>
 <pinref part="R28" gate="G$1" pin="2"/>
-</segment>
-<segment>
+<pinref part="R3" gate="G$1" pin="1"/>
+<wire x1="144.78" y1="73.66" x2="147.32" y2="73.66" width="0.1524" layer="91"/>
+<junction x="144.78" y="73.66"/>
+</segment>
+<segment>
